File: Electronics/TeensyServoController.sch (EAGLE design)
At the start: 17 parts, among them U1 MK20DX128VLH5, U2 AP3211_SWITCHING_REGULATOR, U3 AP3211_SWITCHING_REGULATOR, U4 AP3211_SWITCHING_REGULATOR

Commit message: Continued Work on Teensy servo controller
Parts:
- added C1, C5, C6: 10nF, resistor:C-EUC0402
- added C10, C11, C12, C14, C15, C16, C7, C8: 0.1uF, resistor:C-EUC0402
- added C13, C9: 2.2uF, resistor:C-EUC0603
- added C2, C3, C4: 10uF, resistor:C-EUC0805
- added Q1: 16MHz, crystal:CRYSTALCTS406
- added R1, R3, R4: 349k, resistor:R-US_R0402
- added R2, R5, R6: 49.9k, resistor:R-US_R0402
- added R7, R8: 33, resistor:R-US_R0402
- added R9: 470, resistor:R-US_R0402
- added U5: (no value), SparkFun-Connectors:USB-AB
Connections:
- removed net N$8: U$3.P1.4, U$3.P2.5, U$3.VSS
- new net N$10: R7.1, U5.D-
- new net N$14: C1.2, U2.BS
- new net N$15: R8.2, U1.USB0_DP
- new net N$16: R4.1, R6.2, U4.FB
- new net N$17: C5.2, U3.BS
- new net N$18: R3.1, R5.2, U3.FB
- new net N$19: C6.2, U4.BS
- new net N$20: C6.1, L3.1, R4.2, U4.SW
- new net N$21: C14.1, Q1.2, U1.PTA18
- new net N$22: C15.1, Q1.1, U1.PTA19
- new net N$23: C16.2, U1.VREGIN
- new net N$24: C9.1, R9.1, U1.VDDA
- new net N$25: C7.2, C8.2, C9.2, U1.VREFL, U1.VSSA
- new net N$26: C7.1, U1.VREF_OUT
- new net N$27: C8.1, R9.2, U1.VREFH
- new net N$30: U$3.P3.2, U1.RESET_B
- new net N$31: C10.1, C11.1, C12.1, C13.1, U$3.AVDD, U$3.VDD, U1.VDD, U1.VOUT33
- new net N$6: R1.1, R2.2, U2.FB
- new net N$9: R8.1, U5.D+
- net GND: now also C10.2, C11.2, C12.2, C13.2, C14.2, C15.2, C16.1, C2.2, C3.2, C4.2, R2.1, R5.1, R6.1, U$3.AVSS, U$3.P1.4, U$3.P2.5, U$3.VSS, U1.VSS, U2.GND, U3.GND, U4.GND, U5.GND
- net N$1: now also U5.USBID
- net N$11: now also C5.1, R3.2
- net N$12: now also R7.2, U1.USB0_DM; no longer L3.1, U4.SW
- net N$13: now also C1.1, R1.2
- net VCC: now also C2.1, C3.1, C4.1
Other:
- note added: "349k = 6.5v 257k = 5.5v"
- moved on the sheet: L1, L2, L3, U$3, U1, U2, U3

Commit message: Servo controller mostly done (no I sense)
Parts:
- removed C10, C11, C12, C14, C15, C16: 0.1uF, resistor:C-EUC0402
- removed C13, C9: 2.2uF, resistor:C-EUC0603
- removed Q1: 16MHz, crystal:CRYSTALCTS406
- removed U$3: MINI54TAN, TeensyCustom:MINI54TAN
- added JP10: (no value), SparkFun-Connectors:M02PTH
- added JP11: 3-PIN_JST_ZH_PTH_CONNECTORRIGHT_ANGLE_PTH, My Parts:3-PIN_JST_ZH_PTH_CONNECTORRIGHT_ANGLE_PTH
- added JP12: (no value), SparkFun-Connectors:M03X22X3_SILK_SM
- added R10, R11, R12, R17, R20, R23: 1k, resistor:R-US_R0402
- added R13, R14, R15, R18, R21, R24: 63.4k, resistor:R-US_R0402
- added R16, R19, R22: 0.1, resistor:R-US_R0805
- added U6, U7, U8: MCP6L02T-E/MS, linear:MCP602ST
- C7: value 0.1uF -> 10uF; device resistor:C-EUC0402 -> resistor:C-EUC0805
- JP1, JP2, JP3, JP4, JP5, JP6, JP7, JP8, JP9: device SparkFun-Connectors:M04LOCK -> SparkFun-Connectors:M04PTH
- L1, L2, L3: device SparkFun-Passives:INDUCTORCR75 -> inductors:INDUCTOR
- R7, R8: value 33 -> 0.1; device resistor:R-US_R0402 -> resistor:R-US_R0805
- R9: value 470 -> 0.1; device resistor:R-US_R0402 -> resistor:R-US_R0805
- U1: value MK20DX128VLH5 -> TEENSY_3.1_ALLPINS; device TeensyCustom:MK20DX128VLH5 -> Teensy3.0:TEENSY_3.1_ALLPINS
- U2, U3, U4: value AP3211_SWITCHING_REGULATOR -> AP3211KTR-G1
- U5: value (none) -> AP2210N-3.3TRG1; device SparkFun-Connectors:USB-AB -> My Parts:AP7313SOT23R
Connections:
- removed net N$1: U$3.P0.0, U1.PTA1, U5.USBID
- removed net N$12: R7.2, U1.USB0_DM
- removed net N$15: R8.2, U1.USB0_DP
- removed net N$21: C14.1, Q1.2, U1.PTA18
- removed net N$22: C15.1, Q1.1, U1.PTA19
- removed net N$23: C16.2, U1.VREGIN
- removed net N$24: C9.1, R9.1, U1.VDDA
- removed net N$25: C7.2, C8.2, C9.2, U1.VREFL, U1.VSSA
- removed net N$26: C7.1, U1.VREF_OUT
- removed net N$27: C8.1, R9.2, U1.VREFH
- removed net N$30: U$3.P3.2, U1.RESET_B
- removed net N$31: C10.1, C11.1, C12.1, C13.1, U$3.AVDD, U$3.VDD, U1.VDD, U1.VOUT33
- removed net N$4: U$3.P0.1, U1.PTA2
- new net CS0: JP12.3, U1.10/TX2/CS0/PWM
- new net CURRENT-1: JP1.1, R7.2, U6A.+IN
- new net CURRENT-3: JP3.1, R8.2, U6B.+IN
- new net CURRENT-4: JP4.1, R9.2, U7A.+IN
- new net CURRENT-6: JP6.1, R16.2, U7B.+IN
- new net CURRENT-7: JP7.1, R19.2, U8A.+IN
- new net CURRENT-9: JP9.1, R22.2, U8B.+IN
- new net EN-1: U1.33, U2.EN
- new net EN-2: U1.24, U3.EN
- new net EN-3: U1.32/PWM, U4.EN
- new net MISO/MOSI: JP12.5, U1.12/MISO
- new net MOSI/MISO: JP12.6, U1.11/MOSI
- new net SAT-RX: JP10.1, JP11.3, U1.0/RX1
- new net SCLK: JP12.4, U1.13/SCK/LED
- new net SENSE-1: R13.2, U6A.OUT
- new net SENSE-3: R14.2, U6B.OUT
- new net SENSE-4: R15.2, U7A.OUT
- new net SENSE-6: R18.2, U7B.OUT
- new net SENSE-7: R21.2, U8A.OUT
- new net SENSE-9: R24.2, U8B.OUT
- new net VDD: C8.1, JP11.1, U1.3.3V, U1.AREF, U1.VIN, U5.VOUT, U6P.V+, U7P.V+, U8P.V+
- net ANALOG-1: now also U1.22/A8/PWM
- net ANALOG-2: now also U1.21/A7/CS3/PWM
- net ANALOG-3: now also U1.20/A6/CS2/PWM
- net ANALOG-4: now also U1.19/A5/SCL
- net ANALOG-5: now also U1.18/A4/SDA0
- net ANALOG-6: now also U1.17/A3
- net ANALOG-7: now also U1.16/A2
- net ANALOG-8: now also U1.15/A1/CS4
- net ANALOG-9: now also U1.14/A0
- net GND: now also C7.2, C8.2, JP10.2, JP11.2, JP12.1, R10.2, R11.2, R12.2, R16.1, R17.2, R19.1, R20.2, R22.1, R23.2, R7.1, R8.1, R9.1, U1.AGND, U1.GND, U6P.V-, U7P.V-, U8P.V-; no longer C10.2, C11.2, C12.2, C13.2, C14.2, C15.2, C16.1, JP1.1, JP3.1, JP4.1, JP6.1, JP7.1, JP9.1, U$3.AVSS, U$3.P1.4, U$3.P2.5, U$3.VSS, U1.VSS
- net N$10: now also R20.1, R21.1, U8A.-IN; no longer R7.1, U5.D-
- net N$2: now also R10.1, R13.1, U6A.-IN; no longer U$3.P0.5, U$3.P0.6, U1.PTA3
- net N$3: now also R11.1, R14.1, U6B.-IN; no longer U$3.P0.7, U1.PTA0
- net N$5: now also R12.1, R15.1, U7A.-IN; no longer U$3.P3.5, U1.PTB2
- net N$7: now also R17.1, R18.1, U7B.-IN; no longer U$3.P3.4, U1.PTB3
- net N$9: now also R23.1, R24.1, U8B.-IN; no longer R8.1, U5.D+
- net SERVO-1: now also U1.1/TX1
- net SERVO-2: now also U1.2
- net SERVO-3: now also U1.3/PWM/CAN-TX
- net SERVO-4: now also U1.4/PWM/CAN-RX
- net SERVO-5: now also U1.5/PWM
- net SERVO-6: now also U1.6/PWM
- net SERVO-7: now also U1.7/RX3
- net SERVO-8: now also U1.8/TX3
- net SERVO-9: now also U1.9/RX2/CS1/PWM
- net VCC: now also C7.1, JP12.2, U5.VIN
Other:
- moved on the sheet: C7, C8, JP4, JP5, JP6, JP7, JP8, JP9, R7, R8, R9

Commit message: Electronics finalized and ordered
Parts:
- removed R21, R24: 63.4k, resistor:R-US_R0402
- removed R22: 0.1, resistor:R-US_R0805
- removed R23: 1k, resistor:R-US_R0402
- added C10, C11, C9: 22uF, resistor:C-EUC0603
- added C12: 10uF, resistor:C-EUC0805
- added C13, C14, C23, C24, C25, C26, C27, C28, C29, C30, C31, C32, C33, C34, C35, C36, C37, C38: 0.1uF, resistor:C-EUC0402
- added C15, C16: 0.1uF, resistor:C-EUC0603
- added C17, C18, C19, C20, C21, C22: 1uF, resistor:C-EUC0603
- added JP14, JP15: (no value), SparkFun-Connectors:M02PTH
- added LED1, LED2: (no value), SparkFun-LED:LED0603
- added TP1, TP2, TP3, TP4, TP5, TP6: TEST-POINT3, SparkFun-Passives:TEST-POINT3
- added U10, U11, U9: (no value), My Parts:TS1102
- added U12, U13: MIC5225, My Parts:MIC5225
- C8: device resistor:C-EUC0402 -> resistor:C-EUC0603
- R10, R11, R12: value 1k -> 0.027; device resistor:R-US_R0402 -> resistor:R-US_R0603
- R13, R14, R15: value 63.4k -> (none)
- R16, R19: value 0.1 -> (none); device resistor:R-US_R0805 -> resistor:R-US_R0603
- R17: value 1k -> (none); device resistor:R-US_R0402 -> resistor:R-US_R0603
- R18: value 63.4k -> (none); device resistor:R-US_R0402 -> resistor:R-US_R0603
- R20: value 1k -> (none)
- R7, R8, R9: value 0.1 -> 0.027; device resistor:R-US_R0805 -> resistor:R-US_R0603
- U6, U7, U8: value MCP6L02T-E/MS -> (none); device linear:MCP602ST -> My Parts:TS1102
Connections:
- removed net N$2: R10.1, R13.1, U6A.-IN
- removed net N$3: R11.1, R14.1, U6B.-IN
- removed net N$5: R12.1, R15.1, U7A.-IN
- removed net SENSE-1: R13.2, U6A.OUT
- removed net SENSE-3: R14.2, U6B.OUT
- removed net SENSE-4: R15.2, U7A.OUT
- removed net SENSE-6: R18.2, U7B.OUT
- removed net SENSE-7: R21.2, U8A.OUT
- removed net SENSE-9: R24.2, U8B.OUT
- new net AREF: C13.1, R16.2, U1.AREF, U12.VOUT
- new net AREF2: C14.1, R18.2, U1.A13, U13.VOUT
- new net BATT_SENSE: C29.1, R14.1, R15.2, U1.28/A17
- new net I2C_SCL: JP14.1, U1.29/A18/SCL1
- new net I2C_SDA: JP15.2, U1.30/A19/SDA1
- new net N$1: LED1.A, R13.1
- new net N$8: R20.2, U1.25/PWM
- new net SERVO-1_VDD: C17.1, JP1.2, R7.2, U6.RS-
- new net SERVO-3_VDD: C18.1, JP3.2, R8.2, U7.RS-
- new net SERVO-4_VDD: C19.1, JP4.2, R9.2, U8.RS-
- new net SERVO-6_VDD: C20.1, JP6.2, R10.2, U9.RS-
- new net SERVO-7_VDD: C21.1, JP7.2, R11.2, U10.RS-
- new net SERVO-9_VDD: C22.1, JP9.2, R12.2, U11.RS-
- net ANALOG-1: now also C30.1
- net ANALOG-2: now also C31.1
- net ANALOG-3: now also C32.1
- net ANALOG-4: now also C33.1
- net ANALOG-5: now also C34.1
- net ANALOG-6: now also C35.1
- net ANALOG-7: now also C36.1
- net ANALOG-8: now also C37.1
- net ANALOG-9: now also C38.1
- net CURRENT-1: now also C23.1, TP1.1, U1.A10, U6.OUT; no longer JP1.1, R7.2, U6A.+IN
- net CURRENT-3: now also C24.1, TP2.1, U1.A11, U7.OUT; no longer JP3.1, R8.2, U6B.+IN
- net CURRENT-4: now also C25.1, TP3.1, U1.A12, U8.OUT; no longer JP4.1, R9.2, U7A.+IN
- net CURRENT-6: now also C26.1, TP4.1, U1.31/A20, U9.OUT; no longer JP6.1, R16.2, U7B.+IN
- net CURRENT-7: now also C27.1, TP5.1, U1.26/A15, U10.OUT; no longer JP7.1, R19.2, U8A.+IN
- net CURRENT-9: now also C28.1, TP6.1, U1.27/A16, U11.OUT; no longer JP9.1, R22.2, U8B.+IN
- net GND: now also C10.2, C11.2, C12.2, C13.2, C14.2, C15.2, C16.2, C17.2, C18.2, C19.2, C20.2, C21.2, C22.2, C23.2, C24.2, C25.2, C26.2, C27.2, C28.2, C29.2, C30.2, C31.2, C32.2, C33.2, C34.2, C35.2, C36.2, C37.2, C38.2, C9.2, JP1.1, JP15.1, JP3.1, JP4.1, JP6.1, JP7.1, JP9.1, LED1.C, LED2.C, R15.1, R17.1, U10.GND, U10.P$1, U11.GND, U11.P$1, U12.GND, U13.GND, U6.GND, U6.P$1, U7.GND, U7.P$1, U8.GND, U8.P$1, U9.GND, U9.P$1; no longer R10.2, R11.2, R12.2, R16.1, R17.2, R20.2, R22.1, R23.2, R7.1, R8.1, R9.1, U6P.V-, U7P.V-, U8P.V-
- net N$10: now also LED2.A; no longer R21.1, U8A.-IN
- net N$7: now also R16.1, R17.2, U12.ADJ; no longer R17.1, R18.1, U7B.-IN
- net N$9: now also R18.1, R19.2, U13.ADJ; no longer R23.1, R24.1, U8B.-IN
- net SERVO_VDD-1: now also C11.1, R7.1, R8.1, U6.RS+, U7.RS+; no longer JP1.2, JP3.2
- net SERVO_VDD-2: now also C10.1, R10.1, R9.1, U8.RS+, U9.RS+; no longer JP4.2, JP6.2
- net SERVO_VDD-3: now also C9.1, R11.1, R12.1, U10.RS+, U11.RS+; no longer JP7.2, JP9.2
- net VCC: now also C12.1, C15.1, C16.1, R14.2, U12.EN, U12.VIN, U13.EN, U13.VIN; no longer JP12.2
- net VDD: now also JP12.2, JP14.2, R13.2; no longer U1.AREF, U6P.V+, U7P.V+, U8P.V+
Other:
- note added: "=[R15/(R14+R15)]*Vcc"
- note added: "Vout=1.24*(1+(Rtop/Rbot)) Rbot must be < 300k"
- moved on the sheet: R10, R11, R12, R13, R14, R15, R16, R17, R18, R19, R20, R7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
